File: IO.kicad_sch (KiCad schematic)
At the start: 16 parts, among them J1 Conn_01x02

Commit message: Corrected USB host/slave resistors. Added REG1 DC-DC stage. Removed X2, added X1.
Parts:
- removed D1: STATUS_LED, LED_SMD:LED_0805_2012Metric_Pad1.15x1.40mm_HandSolder, symbol Device:LED
- removed J1: Conn_01x02, Connector_JST:JST_PH_S2B-PH-K_1x02_P2.00mm_Horizontal, symbol Connector_Generic:Conn_01x02
- removed R2: 100Ohms, Resistor_SMD:R_0402_1005Metric_Pad0.72x0.64mm_HandSolder, symbol Device:R_Small_US
- removed R9: 56kOhms, Resistor_SMD:R_0402_1005Metric_Pad0.72x0.64mm_HandSolder, symbol Device:R_Small_US
- removed USB1: HX TYPE-C 6P LT H5.0, easyeda2kicad:USB-C-SMD_HX-TYPE-C-6P-LT-H5.0, symbol easyeda2kicad:HXTYPE-C6PLTH5.0
- added LED1: SZYY1615RGB-A 4PIN, MyLib:LED-ARRAY-SMD_4P-L1.6-W1.5_SZYY1615RGB-A, symbol MySymbols:SZYY1615RGB-A4PIN
- added R10, R8, R9: R_Small_US, FobitLib:R_0402_1005Metric_Pad0.72x0.64mm_HandSolder, symbol FobitSymbols:R_Small_US
- added R4, R5: 5.1kOhms, FobitLib:R_0402_1005Metric_Pad0.72x0.64mm_HandSolder, symbol FobitSymbols:R_Small_US
- added USB1: TYPE-C16PIN, MyLib:USB-C-SMD_TYPE-C16PIN, symbol MySymbols:TYPE-C16PIN
- C3: renamed from C7; footprint Capacitor_SMD:C_0402_1005Metric_Pad0.74x0.62mm_HandSolder -> FobitLib:C_0402_1005Metric_Pad0.74x0.62mm_HandSolder; symbol Device:C_Small -> FobitSymbols:C_Small
- R1: footprint (none) -> FobitLib:R_0402_1005Metric_Pad0.72x0.64mm_HandSolder; symbol Device:R_Small_US -> FobitSymbols:R_Small_US
- R2: renamed from R3; footprint (none) -> FobitLib:R_0402_1005Metric_Pad0.72x0.64mm_HandSolder; symbol Device:R_Small_US -> FobitSymbols:R_Small_US
- R3: renamed from R4; footprint (none) -> FobitLib:R_0402_1005Metric_Pad0.72x0.64mm_HandSolder; symbol Device:R_Small_US -> FobitSymbols:R_Small_US
- R6: renamed from R5; footprint (none) -> FobitLib:R_0402_1005Metric_Pad0.72x0.64mm_HandSolder; symbol Device:R_Small_US -> FobitSymbols:R_Small_US
- R7: renamed from R6; footprint (none) -> FobitLib:R_0402_1005Metric_Pad0.72x0.64mm_HandSolder; symbol Device:R_Small_US -> FobitSymbols:R_Small_US
- SW_LOCK1, SW_PANIC1, SW_SPECIAL1, SW_START1, SW_UNLOCK1: footprint easyeda2kicad:SW-SMD_4P-L5.2-W5.2-P3.70-LS6.4_UK-B0233XX -> FobitLib:SW-SMD_4P-L5.2-W5.2-P3.70-LS6.4_UK-B0233XX; symbol easyeda2kicad:G4R152312 -> FobitSymbols:G4R152312
Connections:
- net GND: now also LED1.4 (K), R4.1, R5.1, USB1.1 (SHELL), USB1.2 (SHELL), USB1.3 (SHELL), USB1.4 (SHELL), USB1.A1B12 (GND), USB1.B1A12 (GND)
- net USBC_V+: now also USB1.A4B9 (VBUS), USB1.B4A9 (VBUS)
- new net: R4.2, USB1.B5 (CC2)
- new net: R5.2, USB1.A5 (CC1)
- new net: LED1.1 (A), R8.2
- new net: LED1.2 (A), R9.2
- new net: LED1.3 (A), R10.2
- new net SOC_USB_D+: USB1.A6 (DP1), USB1.B6 (DP2)
- new net SOC_USB_D-: USB1.A7 (DN1), USB1.B7 (DN2)
- new net STATUS_LED_B: R10.1
- new net STATUS_LED_G: R9.1
- new net STATUS_LED_R: R8.1
Other:
- moved on the sheet: C3
